File: docs/kicad_STM32F401CCU6_meteostation/debugger_programmer.kicad_sch (KiCad schematic)
At the start: 1 part, among them J1 Generic Programmer

Commit message: docs: Finish M0 Hardware Scheme
Parts:
- removed J1: Generic Programmer, symbol Connector:Conn_ST_STDC14
- added J3: Conn_ARM_SWD, Connector:Tag-Connect_TC2030-IDC-FP_2x03_P1.27mm_Vertical, symbol Connector:Conn_ARM_SWD_TagConnect_TC2030
Connections:
- net GND: now also J3.5 (GND)
- net NRST: now also J3.3 (~{RESET})
- new net +3.3V: J3.1 (VCC)
- new net SWCLK: J3.4 (SWCLK)
- new net SWDIO: J3.2 (SWDIO)
- no-connect marks 7 -> 1
Other:
- title: Programming and Debugging Interfaces Scheme -> Programmer and Debugger Interfaces Scheme
Changed lines of the file:
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@@
   (paper "A5")
   (title_block
-    (title "Programming and Debugging Interfaces Scheme")
+    (title "Programmer and Debugger Interfaces Scheme")
+    (date "2026-10-15")
+    (rev "v1.0")
+    (comment 1 "Any supported debugger and programmer may be used")
   )
-  (no_connect (at 71.12 31.115))
-  (no_connect (at 68.58 66.675))
-  (no_connect (at 83.82 59.055))
-  (no_connect (at 83.82 61.595))
-  (no_connect (at 83.82 53.975))
-  (no_connect (at 83.82 46.355))
-  (no_connect (at 83.82 48.895))
-  (wire (pts (xy 83.82 36.195) (xy 95.885 36.195))
-    (stroke (width 0) (type default))
-  )
-  (wire (pts (xy 83.82 43.815) (xy 95.885 43.815))
-    (stroke (width 0) (type default))
-  )
-  (wire (pts (xy 83.82 41.275) (xy 95.885 41.275))
-    (stroke (width 0) (type default))
-  )
-  (hierarchical_label "NRST" (shape bidirectional) (at 95.885 36.195 0) (fields_autoplaced)
+  (no_connect (at 38.1 38.1))
+  (hierarchical_label "NRST" (shape bidirectional) (at 38.1 27.94 0) (fields_autoplaced)
     (effects (font (size 1.27 1.27)) (justify left))
   )
-  (hierarchical_label "SYS_JTMS_SWDIO" (shape bidirectional) (at 95.885 43.815 0) (fields_autoplaced)
+  (hierarchical_label "SWCLK" (shape bidirectional) (at 38.1 33.02 0) (fields_autoplaced)
     (effects (font (size 1.27 1.27)) (justify left))
   )
-  (hierarchical_label "SYS_JTMS_SWCLK" (shape bidirectional) (at 95.885 41.275 0) (fields_autoplaced)
+  (hierarchical_label "SWDIO" (shape bidirectional) (at 38.1 35.56 0) (fields_autoplaced)
     (effects (font (size 1.27 1.27)) (justify left))
   )
-  (hierarchical_label "GND" (shape bidirectional) (at 71.12 66.675 270) (fields_autoplaced)
-    (effects (font (size 1.27 1.27)) (justify right))
-  )
-  (symbol (lib_id "Connector:Conn_ST_STDC14") (at 71.12 48.895 0) (unit 1)
+  (symbol (lib_id "power:GND") (at 27.94 43.18 0) (mirror y) (unit 1)
     (in_bom yes) (on_board yes) (dnp no) (fields_autoplaced)
-    (property "Reference" "J1" (at 59.69 47.625 0)
-      (effects (font (size 1.27 1.27)) (justify right))
-    )
-    (property "Value" "Generic Programmer " (at 59.69 50.165 0)
-      (effects (font (size 1.27 1.27)) (justify right))
-    )
-    (property "Footprint" "" (at 71.12 48.895 0)
+    (property "Reference" "#PWR09" (at 27.94 49.53 0)
       (effects (font (size 1.27 1.27)) hide)
     )
-    (property "Datasheet" "https://www.st.com/content/ccc/resource/technical/document/user_manual/group1/99/49/91/b6/b2/3a/46/e5/DM00526767/files/DM00526767.pdf/jcr:content/translations/en.DM00526767.pdf" (at 62.23 80.645 90)
+    (property "Value" "GND" (at 27.94 48.26 0)
+      (effects (font (size 1.27 1.27)))
+    )
+    (property "Footprint" "" (at 27.94 43.18 0)
       (effects (font (size 1.27 1.27)) hide)
     )
-    (pin "7")
-    (pin "10")
-    (pin "3")
+    (property "Datasheet" "" (at 27.94 43.18 0)
+      (effects (font (size 1.27 1.27)) hide)
+    )
     (pin "1")
-    (pin "11")
-    (pin "8")
-    (pin "6")
-    (pin "9")
-    (pin "12")
-    (pin "4")
-    (pin "2")
-    (pin "5")
-    (pin "13")
-    (pin "14")
     (instances
       (project "kicad_STM32F401CCU6_meteostation"
         (path "/d357996e-dbf2-4ea9-a910-dce674dbe94c/2b0d3a3f-870c-49a6-9675-ada91808f994"
-          (reference "J1") (unit 1)
+          (reference "#PWR09") (unit 1)
         )
       )
+    )
+  )
+  (symbol (lib_id "Connector:Conn_ARM_SWD_TagConnect_TC2030") (at 30.48 33.02 0) (unit 1)
+    (in_bom no) (on_board yes) (dnp no)
+    (property "Reference" "J3" (at 40.64 45.72 0)
+      (effects (font (size 1.27 1.27)) (justify right))
+    )
+    (property "Value" "Conn_ARM_SWD" (at 46.99 48.26 0)
+      (effects (font (size 1.27 1.27)) (justify right))
+    )
+    (property "Footprint" "Connector:Tag-Connect_TC2030-IDC-FP_2x03_P1.27mm_Vertical" (at 30.48 50.8 0)
+      (effects (font (size 1.27 1.27)) hide)
+    )
+    (property "Datasheet" "https://www.tag-connect.com/wp-content/uploads/bsk-pdf-manager/TC2030-CTX_1.pdf" (at 30.48 48.26 0)
+      (effects (font (size 1.27 1.27)) hide)
+    )
+    (pin "3")
+    (pin "5")
+    (pin "6")
+    (pin "1")
+    (pin "2")
+    (pin "4")
+    (instances
+      (project "kicad_STM32F401CCU6_meteostation"
+        (path "/d357996e-dbf2-4ea9-a910-dce674dbe94c/2b0d3a3f-870c-49a6-9675-ada91808f994"
+          (reference "J3") (unit 1)
+        )
+      )
+    )
+  )
+  (symbol (lib_id "power:+3.3V") (at 27.94 22.86 0) (unit 1)
+    (in_bom yes) (on_board yes) (dnp no) (fields_autoplaced)
+    (property "Reference" "#PWR016" (at 27.94 26.67 0)
+      (effects (font (size 1.27 1.27)) hide)
+    )
+    (property "Value" "+3.3V" (at 27.94 17.78 0)
+      (effects (font (size 1.27 1.27)))
+    )
+    (property "Footprint" "" (at 27.94 22.86 0)
+      (effects (font (size 1.27 1.27)) hide)
+    )
+    (property "Datasheet" "" (at 27.94 22.86 0)
+      (effects (font (size 1.27 1.27)) hide)
+    )
+    (pin "1")
+    (instances
+      (project "kicad_STM32F401CCU6_meteostation"
+        (path "/d357996e-dbf2-4ea9-a910-dce674dbe94c/2b0d3a3f-870c-49a6-9675-ada91808f994"
+          (reference "#PWR016") (unit 1)
+        )
+      )
