File: docs/kicad_STM32F401CCU6_meteostation/kicad_STM32F401CCU6_meteostation.kicad_sch (KiCad schematic)
At the start: 3 parts, among them U2 STM32F401CCUx

Commit message: docs: Finish M0 Hardware Scheme
Parts:
- removed C8: 100nF, symbol Device:C
- removed R1: 10kOm, symbol Device:R
- removed U2: STM32F401CCUx, Package_DFN_QFN:QFN-48-1EP_7x7mm_P0.5mm_EP5.6x5.6mm, symbol MCU_ST_STM32F4:STM32F401CCUx
Other:
- removed sheet power_supply
- added sheet mcu (mcu.kicad_sch)
- sheet communication_interfaces ports: added USART2_RX, USART2_TX; removed none
- sheet debugger_programmer ports: added NRST, SWCLK, SWDIO; removed none
- title: (none) -> Sheets' pins connections
